Commit message: update xacros and launch to work

File: summit_xls_ur5_description/robots/summit_xls_ur5_omni.urdf.xacro (robot description, xacro)
@@ -12,5 +12,5 @@
 	<xacro:property name="hq" value="true" />
 	<!-- Import Summit XL Steel -->
-	<xacro:include filename="$(find summit_xl_description)/robots/summit_xl_hls_omni.urdf.xacro"/>
+	<xacro:include filename="$(find summit_xl_description)/robots/summit_xls_std.urdf.xacro"/>
 	<!-- Import UR5 arm -->
 	<xacro:include filename="$(find ur_description)/urdf/ur5.urdf.xacro" />
@@ -26,9 +26,9 @@
     </joint -->
 	<!-- UR5 Arm -->
-    <xacro:ur5_robot prefix="arm_" joint_limited="true">
+    <xacro:ur5_robot prefix="$(prefix)arm_" joint_limited="true">
     </xacro:ur5_robot>
     <joint name="arm_base_joint" type="fixed">
 		<origin xyz="0.175 0 0.303" rpy="0 0 0" />
-		<parent link="base_link" />
+		<parent link="$(arg prefix)base_link" />
 		<child link="arm_base_link" />
 	</joint>

Commit message: add missing changes; corrections to urdf

File: summit_xls_ur5_description/robots/summit_xls_ur5_omni.urdf.xacro (robot description, xacro)
@@ -26,10 +26,10 @@
     </joint -->
 	<!-- UR5 Arm -->
-    <xacro:ur5_robot prefix="$(prefix)arm_" joint_limited="true">
+    <xacro:ur5_robot prefix="$(arg prefix)arm_" joint_limited="true">
     </xacro:ur5_robot>
-    <joint name="arm_base_joint" type="fixed">
+    <joint name="$(arg prefix)arm_base_joint" type="fixed">
 		<origin xyz="0.175 0 0.303" rpy="0 0 0" />
 		<parent link="$(arg prefix)base_link" />
-		<child link="arm_base_link" />
+		<child link="$(arg prefix)arm_base_link" />
 	</joint>
 </robot>

Commit message: backup gazebo work

File: summit_xls_ur5_description/robots/summit_xls_ur5_omni.urdf.xacro (robot description, xacro)
@@ -8,15 +8,16 @@
 	<xacro:property name="base_arm_x" value="0.175"/>
 	<xacro:property name="base_arm_y" value="0.0"/>
-	<xacro:property name="base_arm_z" value="0.303"/>
+	<xacro:property name="base_arm_z" value="0.3875"/>
 	<!-- Flag to select the high or low quality model -->
 	<xacro:property name="hq" value="true" />
+	<xacro:arg name="ros_planar_move_plugin" default="false"/>
 	<!-- Import Summit XL Steel -->
-	<xacro:include filename="$(find summit_xl_description)/robots/summit_xls_std.urdf.xacro"/>
+	<xacro:include filename="$(find summit_xls_ur5_description)/robots/summit_xls_std.urdf.xacro"/>
 	<!-- Import UR5 arm -->
 	<xacro:include filename="$(find ur_description)/urdf/ur5.urdf.xacro" />
 	<!-- SENSORS -->
-    <!-- xacro:sensor_sick_s300 name="laser_front" parent="base_link">
+    <!-- <xacro:sensor_sick_s300 name="laser_front" parent="base_link">
 		<origin xyz="${front_laser_offset_x} ${front_laser_offset_y} ${front_laser_offset_z}" rpy="0 0 ${-PI/4.0}"/>
-	</xacro:sensor_sick_s300 -->
+	</xacro:sensor_sick_s300> -->
     <!-- xacro:BB2-08S2C-38 frame="bumblebee2" name="bumblebee2" />
 		<joint name="world_camera_joint" type="fixed">
@@ -29,5 +30,5 @@
     </xacro:ur5_robot>
     <joint name="$(arg prefix)arm_base_joint" type="fixed">
-		<origin xyz="0.175 0 0.303" rpy="0 0 0" />
+		<origin xyz="${base_arm_x} ${base_arm_y} ${base_arm_z}" rpy="0 0 0" />
 		<parent link="$(arg prefix)base_link" />
 		<child link="$(arg prefix)arm_base_link" />
